Commit message: feat(so101_bringup): Gazebo Ionic simulation with ros2_control
Add the so101_bringup package to simulate the SO-101 in Gazebo Ionic
(gz-sim 9, vendored by ROS 2 Kilted) with ros2_control:
- worlds/empty.sdf, config/ros2_controllers.yaml
  (joint_state_broadcaster, arm_controller=JTC over the 5 arm joints,
  gripper_controller=parallel_gripper_action_controller over the gripper)
- launch/gazebo.launch.py: spawn from /robot_description, /clock bridge,
  ordered controller spawners (jsb -> arm + gripper), headless option

Also fix so101_description for Gazebo Ionic:
- ros2_control plugin ign_ros2_control/IgnitionSystem ->
  gz_ros2_control/GazeboSimSystem
- new so101.gazebo.xacro loading the gz_ros2_control system plugin
- anchor base_link to world (stops the arm falling in sim, removes the
  KDL "root link with an inertia" warning, gives MoveIt a fixed root)

Verified in sim: 3 controllers active, FollowJointTrajectory goal
reached, gripper ParallelGripperCommand working.

File: so101_description/urdf/so101.ros2_control.xacro (robot description, xacro)
@@ -12,5 +12,5 @@
             </xacro:if>
             <xacro:if value="$(eval mode == 'gazebo')">
-            <plugin>ign_ros2_control/IgnitionSystem</plugin>
+            <plugin>gz_ros2_control/GazeboSimSystem</plugin>
             </xacro:if>
             <xacro:if value="$(eval mode == 'real')">

File: so101_description/urdf/so101.urdf.xacro (robot description, xacro)
@@ -11,9 +11,23 @@
     <xacro:arg name="mode" default="gazebo"/>
     <xacro:arg name="joint_states_gui" default="false"/>
+    <xacro:arg name="controllers_file" default="$(find so101_description)/config/initial_positions.yaml"/>
     <xacro:include filename="$(find so101_description)/urdf/so101.urdf"/>
     <xacro:include filename="$(find so101_description)/urdf/so101.transmission.xacro"/>
+    <!-- Anchor the arm to the world: fixes the KDL "root link with an inertia"
+         warning, keeps the base from falling/sliding in Gazebo, and gives MoveIt
+         a fixed virtual joint root. A table-mounted arm is rigidly fixed anyway. -->
+    <link name="world"/>
+    <joint name="world_to_base" type="fixed">
+        <parent link="world"/>
+        <child link="base_link"/>
+        <origin xyz="0 0 0" rpy="0 0 0"/>
+    </joint>
     <xacro:if value="$(eval not joint_states_gui)">
         <xacro:include filename="$(find so101_description)/urdf/so101.ros2_control.xacro"/>
         <xacro:so101_ros2_control name="RobotSystem" initial_positions_file="$(arg initial_positions_file)"/>
+        <xacro:if value="$(eval mode == 'gazebo')">
+            <xacro:include filename="$(find so101_description)/urdf/so101.gazebo.xacro"/>
+            <xacro:so101_gazebo controllers_file="$(arg controllers_file)"/>
+        </xacro:if>
     </xacro:if>
 </robot>
