Commit message: Make the SO-101 arm reusable via a prefixed xacro macro
Wrap the arm description in a `so101_arm` macro parameterized by `prefix` and
`parent`, so the arm can be mounted on another platform (the LeKiwi mobile base)
without frame name collisions (`base_link`, etc.).

- so101.macro.xacro: new macro (frozen onshape geometry, every link/joint
  prefixed; optional mount joint to `parent`, otherwise the `world` anchor is
  handled by the top-level).
- so101.urdf.xacro: now uses the macro (empty prefix) -> standalone unchanged.
- so101.transmission.xacro / so101.ros2_control.xacro: parameterized by `prefix`.

Backward compatible: the standalone render is semantically identical (links,
joints, origins, axes, limits, ros2_control interfaces, transmissions) in both
Gazebo and MoveIt modes. Prepares the S20 mobile manipulation platform.

Co-Authored-By: Claude Opus 4.8 (1M context) <noreply@anthropic.com>

File: so101_description/urdf/so101.ros2_control.xacro (robot description, xacro)
@@ -1,5 +1,5 @@
 <?xml version="1.0"?>
 <robot xmlns:xacro="http://www.ros.org/wiki/xacro" name="so101">
-    <xacro:macro name="so101_ros2_control" params="name initial_positions_file">
+    <xacro:macro name="so101_ros2_control" params="name initial_positions_file prefix:=''">
         <xacro:property name="initial_positions" value="${xacro.load_yaml(initial_positions_file)['initial_positions']}"/>
         <ros2_control name="${name}" type="system" rw_rate="100">
@@ -18,5 +18,5 @@
             </xacro:if>
           </hardware>
-            <joint name="shoulder_pan">
+            <joint name="${prefix}shoulder_pan">
                 <command_interface name="position"/>
                 <state_interface name="position">
@@ -25,5 +25,5 @@
                 <state_interface name="velocity"/>
             </joint>
-            <joint name="shoulder_lift">
+            <joint name="${prefix}shoulder_lift">
                 <command_interface name="position"/>
                 <state_interface name="position">
@@ -32,5 +32,5 @@
                 <state_interface name="velocity"/>
             </joint>
-            <joint name="elbow_flex">
+            <joint name="${prefix}elbow_flex">
                 <command_interface name="position"/>
                 <state_interface name="position">
@@ -39,5 +39,5 @@
                 <state_interface name="velocity"/>
             </joint>
-            <joint name="wrist_flex">
+            <joint name="${prefix}wrist_flex">
                 <command_interface name="position"/>
                 <state_interface name="position">
@@ -46,5 +46,5 @@
                 <state_interface name="velocity"/>
             </joint>
-            <joint name="wrist_roll">
+            <joint name="${prefix}wrist_roll">
                 <command_interface name="position"/>
                 <state_interface name="position">
@@ -53,5 +53,5 @@
                 <state_interface name="velocity"/>
             </joint>
-            <joint name="gripper">
+            <joint name="${prefix}gripper">
                 <command_interface name="position"/>
                 <state_interface name="position">

File: so101_description/urdf/so101.transmission.xacro (robot description, xacro)
@@ -1,63 +1,65 @@
 <?xml version="1.0"?>
 <robot xmlns:xacro="http://ros.org/wiki/xacro" name="so101">
-    <transmission name="gripper_trans">
+    <xacro:macro name="so101_transmission" params="prefix:=''">
+    <transmission name="${prefix}gripper_trans">
         <type>transmission_interface/SimpleTransmission</type>
-        <joint name="gripper">
+        <joint name="${prefix}gripper">
           <hardwareInterface>hardware_interface/PositionJointInterface</hardwareInterface>
         </joint>
-        <actuator name="motor6">
+        <actuator name="${prefix}motor6">
           <hardwareInterface>hardware_interface/PositionJointInterface</hardwareInterface>
           <mechanicalReduction>1</mechanicalReduction>
         </actuator>
       </transmission>
-    <transmission name="wrist_roll_trans">
+    <transmission name="${prefix}wrist_roll_trans">
         <type>transmission_interface/SimpleTransmission</type>
-        <joint name="wrist_roll">
+        <joint name="${prefix}wrist_roll">
           <hardwareInterface>hardware_interface/PositionJointInterface</hardwareInterface>
         </joint>
-        <actuator name="motor5">
+        <actuator name="${prefix}motor5">
           <hardwareInterface>hardware_interface/PositionJointInterface</hardwareInterface>
           <mechanicalReduction>1</mechanicalReduction>
         </actuator>
       </transmission>
-    <transmission name="wrist_flex_trans">
+    <transmission name="${prefix}wrist_flex_trans">
         <type>transmission_interface/SimpleTransmission</type>
-        <joint name="wrist_flex">
+        <joint name="${prefix}wrist_flex">
           <hardwareInterface>hardware_interface/PositionJointInterface</hardwareInterface>
         </joint>
-        <actuator name="motor4">
+        <actuator name="${prefix}motor4">
           <hardwareInterface>hardware_interface/PositionJointInterface</hardwareInterface>
           <mechanicalReduction>1</mechanicalReduction>
         </actuator>
       </transmission>
-    <transmission name="elbow_flex_trans">
+    <transmission name="${prefix}elbow_flex_trans">
         <type>transmission_interface/SimpleTransmission</type>
-        <joint name="elbow_flex">
+        <joint name="${prefix}elbow_flex">
           <hardwareInterface>hardware_interface/PositionJointInterface</hardwareInterface>
         </joint>
-        <actuator name="motor3">
+        <actuator name="${prefix}motor3">
           <hardwareInterface>hardware_interface/PositionJointInterface</hardwareInterface>
           <mechanicalReduction>1</mechanicalReduction>
         </actuator>
       </transmission>
-    <transmission name="shoulder_lift_trans">
+    <transmission name="${prefix}shoulder_lift_trans">
         <type>transmission_interface/SimpleTransmission</type>
-        <joint name="shoulder_lift">
+        <joint name="${prefix}shoulder_lift">
           <hardwareInterface>hardware_interface/PositionJointInterface</hardwareInterface>
         </joint>
-        <actuator name="motor2">
+        <actuator name="${prefix}motor2">
           <hardwareInterface>hardware_interface/PositionJointInterface</hardwareInterface>
           <mechanicalReduction>1</mechanicalReduction>
         </actuator>
       </transmission>
-    <transmission name="shoulder_pan_trans">
+    <transmission name="${prefix}shoulder_pan_trans">
         <type>transmission_interface/SimpleTransmission</type>
-        <joint name="shoulder_pan">
+        <joint name="${prefix}shoulder_pan">
           <hardwareInterface>hardware_interface/PositionJointInterface</hardwareInterface>
         </joint>
-        <actuator name="motor1">
+        <actuator name="${prefix}motor1">
           <hardwareInterface>hardware_interface/PositionJointInterface</hardwareInterface>
           <mechanicalReduction>1</mechanicalReduction>
         </actuator>
       </transmission>
+    </xacro:macro>
 </robot>

File: so101_description/urdf/so101.urdf.xacro (robot description, xacro)
@@ -12,6 +12,10 @@
     <xacro:arg name="joint_states_gui" default="false"/>
     <xacro:arg name="controllers_file" default="$(find so101_description)/config/initial_positions.yaml"/>
-    <xacro:include filename="$(find so101_description)/urdf/so101.urdf"/>
+    <!-- Bras en macro reutilisable (prefix vide => noms standalone inchanges).
+         La meme macro sert au montage sur la base mobile LeKiwi (prefix 'arm_'). -->
+    <xacro:include filename="$(find so101_description)/urdf/so101.macro.xacro"/>
+    <xacro:so101_arm/>
     <xacro:include filename="$(find so101_description)/urdf/so101.transmission.xacro"/>
+    <xacro:so101_transmission/>
     <!-- Anchor the arm to the world: fixes the KDL "root link with an inertia"
          warning, keeps the base from falling/sliding in Gazebo, and gives MoveIt
